File: pcb/pcb.sch (KiCad schematic (older format))
At the start: 88 parts, among them U1 JM20330, U2 SM2258XT, U3 FlashBGA152, U4 Conn_41PIN, U5 SY8008, U6 SY8008, U7 TX4314, Y1 25MHz, Y2 50MHz

Commit message: First revision freeze
Connections:
- net +3V3: now also U1.20 (MODE2)
- net GND: no longer U1.20 (MODE2)
- no-connect marks 60 -> 58
Changed lines of the file:
@@
 Wire Wire Line
 	5400 3200 5500 3200
-Wire Wire Line
-	5500 3200 5500 3400
 Connection ~ 5500 4000
-Wire Wire Line
-	5400 3400 5500 3400
-Connection ~ 5500 3400
-Wire Wire Line
-	5500 3400 5500 3800
 Wire Wire Line
 	5400 3600 5600 3600
@@
 	5500 3800 5500 4000
 Wire Wire Line
-	5600 3300 5600 3600
+	5600 3300 5600 3400
 $Comp
 L Device:R R?
@@
 Wire Wire Line
 	5400 1500 5800 1500
-NoConn ~ 13000 6200
-NoConn ~ 13000 6300
 $Comp
 L power:GND #PWR0163
@@
 NoConn ~ 8400 5900
 Wire Wire Line
+	7200 7900 8000 7900
+Wire Wire Line
+	7200 7600 8000 7600
+Wire Wire Line
+	7900 2700 8400 2700
+$Comp
+L Mechanical:MountingHole H1
+U 1 1 60B1FFAD
+P 6000 6400
+F 0 "H1" H 6100 6446 50  0000 L CNN
+F 1 "MountingHole" H 6100 6355 50  0000 L CNN
+F 2 "MountingHole:MountingHole_2.2mm_M2_Pad_Via" H 6000 6400 50  0001 C CNN
+F 3 "~" H 6000 6400 50  0001 C CNN
+	1    6000 6400
+	1    0    0    -1
+$EndComp
+Wire Wire Line
+	5500 3200 5500 3800
+Wire Wire Line
+	5400 3400 5600 3400
+Wire Wire Line
 	10900 2500 12000 2500
 Wire Wire Line
@@
 Wire Bus Line
 	3700 1700 3700 4700
-Wire Wire Line
-	7200 7900 8000 7900
-Wire Wire Line
-	7200 7600 8000 7600
-Wire Wire Line
-	7900 2700 8400 2700
-$Comp
-L Mechanical:MountingHole H1
-U 1 1 60B1FFAD
-P 6000 6400
-F 0 "H1" H 6100 6446 50  0000 L CNN
-F 1 "MountingHole" H 6100 6355 50  0000 L CNN
-F 2 "MountingHole:MountingHole_2.2mm_M2_Pad_Via" H 6000 6400 50  0001 C CNN
-F 3 "~" H 6000 6400 50  0001 C CNN
-	1    6000 6400
-	1    0    0    -1
-$EndComp
+Connection ~ 5600 3400
+Wire Wire Line
+	5600 3400 5600 3600
 $EndSCHEMATC
